File: Kicad/Revision B1 Parity/16MB SIPPM 30 rev B1.kicad_pcb (KiCad board)
At the start: 4 copper layers, 88.9 x 19.2 mm, 17 parts, among them J1 SIMM-30, U1 MT4LC16M4H9, U2 MT4LC16M4H9, U3 AMS1117-3.3, U4 HM5116100S

Commit message: minor Rev B1 cleanups - not prod ready
Connections:
- J1 pad 24: /2A11 -> /SIMM_A11
Routing:
- net /SIMM_A11: track 5.86 -> 23.0 mm, vias 0 -> 1
- net /2A11: track 82.2 -> 71.2 mm, vias 1 -> 2
- net +3V3: track 15.3 -> 18.1 mm
- net /~{WE}: track 64.8 -> 67.3 mm
- net /2A6: track 65.8 -> 68.3 mm
- net /2A10: track 70.5 -> 72.7 mm
- net GND: track 17.8 -> 20.0 mm
- net /2A4: track 61.9 -> 63.7 mm
- net /VDD_PAR: track 29.0 -> 30.7 mm
- net /2A3: track 77.7 -> 79.4 mm
- net /2A9: track 100.8 -> 102.3 mm
- net /QP: track 18.9 -> 20.4 mm
- net /DP: track 27.3 -> 28.7 mm
- net /2A2: track 65.2 -> 66.5 mm
- net /2A8: track 71.3 -> 72.6 mm
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