File: Kicad/Revision B1 Parity/16MB SIPPM 30 rev B1.kicad_sch (KiCad schematic)
At the start: 16 parts, among them J1 SIMM-30, U1 MT4LC16M4H9, U2 MT4LC16M4H9, U3 AMS1117-3.3, U4 HM5116100S

Commit message: minor Rev B1 cleanups - not prod ready
Connections:
- net 1A11: no longer J1.24 (A11)
- net SIMM_A11: now also J1.24 (A11)
Changed lines of the file:
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@@
-    (effects (font (size 1.27 1.27)) (justify left bottom))
-  )
-  (label "A11" (at 66.04 91.44 0)
     (effects (font (size 1.27 1.27)) (justify left bottom))
   )
   (label "2A6" (at 215.265 74.93 0)
     (effects (font (size 1.27 1.27)) (justify left bottom))
+  )
+  (label "SIMM_A11" (at 66.04 91.44 180)
+    (effects (font (size 1.27 1.27)) (justify right bottom))
   )
   (label "A8" (at 66.04 83.82 0)
@@
   )
   (symbol (lib_id "edge connectors:SIMM-30") (at 86.36 83.82 0) (unit 1)
-    (in_bom yes) (on_board yes) (fields_autoplaced)
-    (property "Reference" "J1" (id 0) (at 88.3794 25.1259 0)
+    (in_bom yes) (on_board yes)
+    (property "Reference" "J1" (id 0) (at 83.82 38.1 0)
       (effects (font (size 1.524 1.524)) (justify left))
     )
-    (property "Value" "SIMM-30" (id 1) (at 88.3794 28.1193 0)
+    (property "Value" "SIMM-30" (id 1) (at 83.82 41.0934 0)
       (effects (font (size 1.524 1.524)) (justify left))
     )
